File: Hardware/PrototypV1_tx/PrototypV1_tx.sch (KiCad schematic (older format))
At the start: 67 parts, among them IC1 STM32L4Q5CGT6, IC2 LD1117V33, J1 FLASH, J10 HC12, J11 WS2812, J12 Conn_01x02_Male, J13 Conn_01x10_Male, J14 Conn_01x07_Male, J15 Conn_01x01_Male, J16 Conn_01x01_Male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

Commit message: Naprawiono błąd z zapisem danych
Parts:
- IC1: symbol STM32L4Q5CGT6:STM32L4Q5CGT6 -> PrototypV1_tx-rescue:STM32L4Q5CGT6-STM32L4Q5CGT6
- IC2: symbol LD1117V33:LD1117V33 -> PrototypV1_tx-rescue:LD1117V33-LD1117V33
- Y1: symbol ABS25-32.768KHZ-6-T:ABS25-32.768KHZ-6-T -> PrototypV1_tx-rescue:ABS25-32.768KHZ-6-T-ABS25-32.768KHZ-6-T
Changed lines of the file:
@@
 $EndDescr
 $Comp
-L STM32L4Q5CGT6:STM32L4Q5CGT6 IC1
+L PrototypV1_tx-rescue:STM32L4Q5CGT6-STM32L4Q5CGT6 IC1
 U 1 1 62DD139C
 P 6000 5900
@@
 DC IN
 $Comp
-L LD1117V33:LD1117V33 IC2
+L PrototypV1_tx-rescue:LD1117V33-LD1117V33 IC2
 U 1 1 62DE1B2A
 P 6300 800
@@
 Connection ~ 8950 900
 $Comp
-L ABS25-32.768KHZ-6-T:ABS25-32.768KHZ-6-T Y1
+L PrototypV1_tx-rescue:ABS25-32.768KHZ-6-T-ABS25-32.768KHZ-6-T Y1
 U 1 1 62EAA395
 P 11400 2100
